File: CC2544 Veriifcation.kicad_sch (KiCad schematic)
At the start: 24 parts

Commit message: release_v1.0
Parts:
- added C11, C13, C15, C17, C19, C20, C4, C5, C6: 100nF, Capacitor_SMD:C_0402_1005Metric, symbol Device:C_Small
- added C22: 220pF, Capacitor_SMD:C_0402_1005Metric, symbol Device:C_Small
- added FID1, FID2, FID3, FID4, FID5, FID6: Fiducial, Fiducial:Fiducial_0.5mm_Mask1.5mm, symbol Mechanical:Fiducial
- added H1, H2, H3, H4: MountingHole, MountingHole:MountingHole_2.7mm_M2.5_DIN965, symbol Mechanical:MountingHole
- added J2: Conn_01x10_Male, Connector_PinHeader_2.54mm:PinHeader_1x10_P2.54mm_Vertical, symbol Connector:Conn_01x10_Male
- C1, C10, C12, C14, C16, C18, C2, C21, C3, C7, C8, C9: renamed from C?; footprint (none) -> Capacitor_SMD:C_0402_1005Metric
- J1: renamed from J?; footprint (none) -> Connector_USB:USB_Micro-B_Molex-105017-0001
- J3: renamed from J?; value Conn_Coaxial -> Atenna; footprint (none) -> Connector_Coaxial:SMA_Amphenol_132134-11_Vertical
- L1, L2, L3, L4: renamed from L?; footprint (none) -> Inductor_SMD:L_0402_1005Metric
- R1, R2, R3, R4: renamed from R?; footprint (none) -> Resistor_SMD:R_0402_1005Metric
- U1: renamed from U?; footprint (none) -> Package_DFN_QFN:QFN-32-1EP_5x5mm_P0.5mm_EP3.45x3.45mm
- Y1: renamed from Y?; footprint (none) -> Crystal:Crystal_SMD_1612-4Pin_1.6x1.2mm
Connections:
- net GND: now also C11.2, C13.2, C15.2, C17.2, C19.2, C20.2, C22.2, C4.2, C5.2, C6.2, J2.10 (Pin_10)
- net +3V3: now reaches C9.1, U1.4 (DCOUPL2)
- net +3V3: now also U1.12 (IOVDD2), U1.16 (AVDD2), U1.19 (AVDD3), U1.22 (AVDD4), U1.23 (AVDD5), U1.24 (AVDD6), U1.26 (AVDD_GUARD), U1.3 (AVDD1), U1.30 (IOVDD3), U1.8 (IOVDD1), C11.1, C13.1, C15.1, C17.1, C19.1, C20.1, C22.1, C4.1, C5.1, C6.1
- net at C1.1, R3.2: now also U1.2 (USB_N); no longer U1.3 (USB_P)
- net at C2.1, R2.2: now also U1.1 (USB_P); no longer U1.2 (USB_N)
- net at U1.10 (P0_1): now also J2.2 (Pin_2)
- net at U1.13 (P0_2): now also J2.3 (Pin_3)
- net at U1.14 (P0_3): now also J2.4 (Pin_4)
- net at U1.15 (RESET_N): now also J2.9 (Pin_9)
- net at U1.28 (P1_2): now also J2.7 (Pin_7)
- net at U1.29 (P1_3): now also J2.8 (Pin_8)
- net at U1.6 (P1_0): now also J2.5 (Pin_5)
- net at U1.7 (P1_1): now also J2.6 (Pin_6)
- net at U1.9 (P0_0): now also J2.1 (Pin_1)
Other:
- moved on the sheet: C16, C18, L1, L2, U1
