File: CC2544 Veriifcation.kicad_pcb (KiCad board)
At the start: 4 copper layers, 40.6 x 40.6 mm, 46 parts, among them J1 USB_B_Mini, J2 Conn_01x10_Male, J3 Atenna, U1 CC2544, Y1 32.000MHz

Commit message: add GPIO silkscreen
Other:
- board text added: "P0_0"
- board text added: "P0_1"
- board text added: "P0_2"
- board text added: "P0_3"
- board text added: "P1_0"
- board text added: "P1_1"
- board text added: "P1_2"
- board text added: "P1_3"
- board text added: "RESET_N"
